File: FFC_Breakout.kicad_pcb (KiCad board)
At the start: 2 copper layers, 22.9 x 17.8 mm, 3 parts, among them J1 LEFT, J2 RIGHT

Commit message: intercept
Parts:
- removed FFC10: FFC_10, Connector_FFC-FPC:Molex_52892-1033_1x10-1MP_P0.5mm_Horizontal
- added J3: FFC_10, Connector_FFC-FPC:Molex_52892-1033_1x10-1MP_P0.5mm_Horizontal, B.Cu at (141.0, 102.2)
- added J4: FFC_10, Connector_FFC-FPC:Molex_52892-1033_1x10-1MP_P0.5mm_Horizontal, F.Cu at (141.0, 111.1)
Routing:
- net Net-(J2-Pad5): track 6.92 -> 15.9 mm, vias 0 -> 1
- net Net-(J1-Pad1): track 7.02 -> 14.9 mm, vias 0 -> 1
- net Net-(J2-Pad4): track 8.23 -> 16.0 mm, vias 0 -> 1
- net Net-(J1-Pad2): track 8.69 -> 16.1 mm, vias 0 -> 1
- net Net-(J1-Pad3): track 13.4 -> 15.8 mm, vias 0 -> 1
- net Net-(J2-Pad3): track 13.5 -> 15.7 mm, vias 0 -> 1
- net Net-(J1-Pad4): track 13.6 -> 15.7 mm, vias 0 -> 1
- net Net-(J2-Pad2): track 13.5 -> 15.4 mm, vias 0 -> 1
- net Net-(J1-Pad5): track 15.2 -> 16.1 mm, vias 0 -> 1
- net Net-(J2-Pad1): track 15.2 -> 15.9 mm, vias 0 -> 1
